File: kicad-files/legshark65.kicad_sch (KiCad schematic)
At the start: 158 parts, among them J1 ARM JTAG, SW1 K2-1187SQ-A4SW-06, SW2 PCM12SMTR, T2 53261-0471, U1 STM32F411CEU6, U3 AT24C256C-SSHL-T, Y1 TAXM8M4RFDCET2T

Commit message: Fixing up the schematic's of daughter and mother boards
Parts:
- D_0, D_1, D_10, D_11, D_12, D_13, D_14, D_15, D_16, D_17, D_18, D_19, D_2, D_20, D_21, D_22, D_23, D_24, D_25, D_26, D_27, D_28, D_29, D_3, D_30, D_31, D_32, D_33, D_34, D_35, D_36, D_37, D_38, D_39, D_4, D_40, D_41, D_42, D_43, D_44, D_45, D_46, D_47, D_48, D_49, D_5, D_50, D_51, D_52, D_53, D_54, D_55, D_56, D_57, D_58, D_59, D_6, D_60, D_61, D_62, D_63, D_64, D_7, D_8, D_9: value D -> 1N4148W
Other:
- moved on the sheet: C9
