File: kicad-files/daughter_board.kicad_sch (KiCad schematic)
At the start: 20 parts, among them J1 TYPE-C-31-M-12, J2 Conn_01x02, T1 53261-0471, U1 TPD4E05U06DQAR, U2 MCP1700T-3302E/TT

Commit message: Updated small things on daughter board bom
Parts:
- FB1: Vendor Part Number (none) -> LCSC C1017
Changed lines of the file:
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@@
+      (effects (font (size 1.27 1.27)) hide)
+    )
+    (property "Vendor Part Number" "LCSC C1017" (at 142.494 149.606 0)
       (effects (font (size 1.27 1.27)) hide)
     )
