File: kicad-files/legshark65_rev2.kicad_pcb (KiCad board)
At the start: 2 copper layers, 285.8 x 93.9 mm, 193 parts, among them J1 ARM JTAG, J2 Conn_01x04, SW1 K2-1187SQ-A4SW-06, SW2 PCM12SMTR, T2 53261-0471, U1 STM32F411CEU6, U2 MCP1700T-3302E/TT, U3 AT24C256C-SSHL-T, Y1 TAXM8M4RFDCET2T

Commit message: Added alternate mods to the right side
Parts:
- added K_75: KEYSW, MX_Only:MXOnly-1.5U-NoLED, F.Cu at (252.4, 85.7)
- added K_82: KEYSW, MX_Only:MXOnly-1U-NoLED, F.Cu at (228.6, 85.7)
- added K_83: KEYSW, MX_Only:MXOnly-1.5U-NoLED, F.Cu at (204.8, 85.7)
- moved J1 39.9 mm to (176.2, 138.1)
- moved J2 38.5 mm to (183.4, 135.7)
- moved D_61 23.8 mm to (40.5, 88.1)
- moved D_60 19.1 mm to (21.4, 88.1)
- moved D_66 14.3 mm to (192.9, 88.1)
- moved D_67 14.3 mm to (211.9, 88.1)
Changed lines of the file:
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@@
       (net 34 "Net-(D_6-A)") (pinfunction "ROW") (pintype "passive"))
   )
+  (footprint "MX_Only:MXOnly-1U-NoLED" (layer "F.Cu")
+    (at 228.6 85.725)
+    (property "Sheetfile" "legshark65_rev2.kicad_sch")
+    (property "Sheetname" "")
+    (attr through_hole)
+    (fp_text reference "K_82" (at 0 3.175) (layer "Dwgs.User")
+        (effects (font (size 1 1) (thickness 0.15)))
+    )
+    (fp_text value "KEYSW" (at 0 -7.9375) (layer "Dwgs.User")
+        (effects (font (size 1 1) (thickness 0.15)))
+    )
+    (fp_line (start -9.525 -9.525) (end 9.525 -9.525)
+      (stroke (width 0.15) (type solid)) (layer "Dwgs.User"))
+    (fp_line (start -9.525 9.525) (end -9.525 -9.525)
+      (stroke (width 0.15) (type solid)) (layer "Dwgs.User"))
+    (fp_line (start -7 -7) (end -7 -5)
+      (stroke (width 0.15) (type solid)) (layer "Dwgs.User"))
+    (fp_line (start -7 5) (end -7 7)
+      (stroke (width 0.15) (type solid)) (layer "Dwgs.User"))
+    (fp_line (start -7 7) (end -5 7)
+      (stroke (width 0.15) (type solid)) (layer "Dwgs.User"))
+    (fp_line (start -5 -7) (end -7 -7)
+      (stroke (width 0.15) (type solid)) (layer "Dwgs.User"))
+    (fp_line (start 5 -7) (end 7 -7)
+      (stroke (width 0.15) (type solid)) (layer "Dwgs.User"))
+    (fp_line (start 5 7) (end 7 7)
+      (stroke (width 0.15) (type solid)) (layer "Dwgs.User"))
+    (fp_line (start 7 -7) (end 7 -5)
+      (stroke (width 0.15) (type solid)) (layer "Dwgs.User"))
+    (fp_line (start 7 7) (end 7 5)
+      (stroke (width 0.15) (type solid)) (layer "Dwgs.User"))
+    (fp_line (start 9.525 -9.525) (end 9.525 9.525)
+      (stroke (width 0.15) (type solid)) (layer "Dwgs.User"))
+    (fp_line (start 9.525 9.525) (end -9.525 9.525)
+      (stroke (width 0.15) (type solid)) (layer "Dwgs.User"))
+    (pad "" np_thru_hole circle (at -5.08 0 48.0996) (size 1.75 1.75) (drill 1.75) (layers "*.Cu" "*.Mask"))
+    (pad "" np_thru_hole circle (at 0 0) (size 3.9878 3.9878) (drill 3.9878) (layers "*.Cu" "*.Mask"))
+    (pad "" np_thru_hole circle (at 5.08 0 48.0996) (size 1.75 1.75) (drill 1.75) (layers "*.Cu" "*.Mask"))
+    (pad "1" thru_hole circle (at -3.81 -2.54) (size 2.25 2.25) (drill 1.47) (layers "*.Cu" "B.Mask")
+      (net 13 "col12") (pinfunction "COL") (pintype "passive"))
+    (pad "2" thru_hole circle (at 2.54 -5.08) (size 2.25 2.25) (drill 1.47) (layers "*.Cu" "B.Mask")
+      (net 96 "Net-(D_68-A)") (pinfunction "ROW") (pintype "passive"))
+  )
   (footprint "MX_Only:MXOnly-1U-NoLED" locked (layer "F.Cu")
     (at 85.725 66.675)
@@
       (net 77 "Net-(D_49-A)") (pinfunction "ROW") (pintype "passive"))
   )
+  (footprint "MX_Only:MXOnly-1.5U-NoLED" (layer "F.Cu")
+    (at 252.4125 85.725)
+    (property "Sheetfile" "legshark65_rev2.kicad_sch")
+    (property "Sheetname" "")
+    (attr through_hole)
+    (fp_text reference "K_75" (at 0 3.175) (layer "Dwgs.User")
+        (effects (font (size 1 1) (thickness 0.15)))
+    )
+    (fp_text value "KEYSW" (at 0 -7.9375) (layer "Dwgs.User")
+        (effects (font (size 1 1) (thickness 0.15)))
+    )
+    (fp_line (start -14.2875 -9.525) (end 14.2875 -9.525)
+      (stroke (width 0.15) (type solid)) (layer "Dwgs.User"))
+    (fp_line (start -14.2875 9.525) (end -14.2875 -9.525)
+      (stroke (width 0.15) (type solid)) (layer "Dwgs.User"))
+    (fp_line (start -14.2875 9.525) (end 14.2875 9.525)
+      (stroke (width 0.15) (type solid)) (layer "Dwgs.User"))
+    (fp_line (start -7 -7) (end -7 -5)
+      (stroke (width 0.15) (type solid)) (layer "Dwgs.User"))
+    (fp_line (start -7 5) (end -7 7)
+      (stroke (width 0.15) (type solid)) (layer "Dwgs.User"))
+    (fp_line (start -7 7) (end -5 7)
+      (stroke (width 0.15) (type solid)) (layer "Dwgs.User"))
+    (fp_line (start -5 -7) (end -7 -7)
+      (stroke (width 0.15) (type solid)) (layer "Dwgs.User"))
+    (fp_line (start 5 -7) (end 7 -7)
+      (stroke (width 0.15) (type solid)) (layer "Dwgs.User"))
+    (fp_line (start 5 7) (end 7 7)
+      (stroke (width 0.15) (type solid)) (layer "Dwgs.User"))
+    (fp_line (start 7 -7) (end 7 -5)
+      (stroke (width 0.15) (type solid)) (layer "Dwgs.User"))
+    (fp_line (start 7 7) (end 7 5)
+      (stroke (width 0.15) (type solid)) (layer "Dwgs.User"))
+    (fp_line (start 14.2875 -9.525) (end 14.2875 9.525)
+      (stroke (width 0.15) (type solid)) (layer "Dwgs.User"))
+    (pad "" np_thru_hole circle (at -5.08 0 48.0996) (size 1.75 1.75) (drill 1.75) (layers "*.Cu" "*.Mask"))
+    (pad "" np_thru_hole circle (at 0 0) (size 3.9878 3.9878) (drill 3.9878) (layers "*.Cu" "*.Mask"))
+    (pad "" np_thru_hole circle (at 5.08 0 48.0996) (size 1.75 1.75) (drill 1.75) (layers "*.Cu" "*.Mask"))
+    (pad "1" thru_hole circle (at -3.81 -2.54) (size 2.25 2.25) (drill 1.47) (layers "*.Cu" "B.Mask")
+      (net 14 "col13") (pinfunction "COL") (pintype "passive"))
+    (pad "2" thru_hole circle (at 2.54 -5.08) (size 2.25 2.25) (drill 1.47) (layers "*.Cu" "B.Mask")
+      (net 97 "Net-(D_69-A)") (pinfunction "ROW") (pintype "passive"))
+  )
   (footprint "MX_Only:MXOnly-1U-NoLED" locked (layer "F.Cu")
     (at 180.975 9.525)
@@
       (net 87 "Net-(D_59-A)") (pinfunction "ROW") (pintype "passive"))
   )
+  (footprint "MX_Only:MXOnly-1.5U-NoLED" (layer "F.Cu")
+    (at 204.7875 85.725)
+    (property "Sheetfile" "legshark65_rev2.kicad_sch")
+    (property "Sheetname" "")
+    (attr through_hole)
+    (fp_text reference "K_83" (at 0 3.175) (layer "Dwgs.User")
+        (effects (font (size 1 1) (thickness 0.15)))
+    )
+    (fp_text value "KEYSW" (at 0 -7.9375) (layer "Dwgs.User")
+        (effects (font (size 1 1) (thickness 0.15)))
+    )
+    (fp_line (start -14.2875 -9.525) (end 14.2875 -9.525)
+      (stroke (width 0.15) (type solid)) (layer "Dwgs.User"))
+    (fp_line (start -14.2875 9.525) (end -14.2875 -9.525)
+      (stroke (width 0.15) (type solid)) (layer "Dwgs.User"))
+    (fp_line (start -14.2875 9.525) (end 14.2875 9.525)
+      (stroke (width 0.15) (type solid)) (layer "Dwgs.User"))
+    (fp_line (start -7 -7) (end -7 -5)
+      (stroke (width 0.15) (type solid)) (layer "Dwgs.User"))
+    (fp_line (start -7 5) (end -7 7)
+      (stroke (width 0.15) (type solid)) (layer "Dwgs.User"))
+    (fp_line (start -7 7) (end -5 7)
+      (stroke (width 0.15) (type solid)) (layer "Dwgs.User"))
+    (fp_line (start -5 -7) (end -7 -7)
+      (stroke (width 0.15) (type solid)) (layer "Dwgs.User"))
+    (fp_line (start 5 -7) (end 7 -7)
+      (stroke (width 0.15) (type solid)) (layer "Dwgs.User"))
+    (fp_line (start 5 7) (end 7 7)
+      (stroke (width 0.15) (type solid)) (layer "Dwgs.User"))
+    (fp_line (start 7 -7) (end 7 -5)
+      (stroke (width 0.15) (type solid)) (layer "Dwgs.User"))
+    (fp_line (start 7 7) (end 7 5)
+      (stroke (width 0.15) (type solid)) (layer "Dwgs.User"))
+    (fp_line (start 14.2875 -9.525) (end 14.2875 9.525)
+      (stroke (width 0.15) (type solid)) (layer "Dwgs.User"))
+    (pad "" np_thru_hole circle (at -5.08 0 48.0996) (size 1.75 1.75) (drill 1.75) (layers "*.Cu" "*.Mask"))
+    (pad "" np_thru_hole circle (at 0 0) (size 3.9878 3.9878) (drill 3.9878) (layers "*.Cu" "*.Mask"))
+    (pad "" np_thru_hole circle (at 5.08 0 48.0996) (size 1.75 1.75) (drill 1.75) (layers "*.Cu" "*.Mask"))
+    (pad "1" thru_hole circle (at -3.81 -2.54) (size 2.25 2.25) (drill 1.47) (layers "*.Cu" "B.Mask")
+      (net 11 "col10") (pinfunction "COL") (pintype "passive"))
+    (pad "2" thru_hole circle (at 2.54 -5.08) (size 2.25 2.25) (drill 1.47) (layers "*.Cu" "B.Mask")
+      (net 94 "Net-(D_66-A)") (pinfunction "ROW") (pintype "passive"))
+  )
   (footprint "MX_Only:MXOnly-1U-NoLED" locked (layer "F.Cu")
     (at 66.675 85.725)
@@
   )
   (footprint "Diode_SMD:D_SOD-523" (layer "B.Cu")
-    (at 207.16875 88.10625 90)
+    (at 192.88125 88.10625 90)
     (descr "http://www.diodes.com/datasheets/ap02001.pdf p.144")
     (tags "Diode SOD523")
@@
   )
   (footprint "Diode_SMD:D_SOD-523" (layer "B.Cu")
-    (at 40.48125 88.10625 90)
+    (at 21.43125 88.10625 90)
     (descr "http://www.diodes.com/datasheets/ap02001.pdf p.144")
     (tags "Diode SOD523")
@@
   )
   (footprint "Diode_SMD:D_SOD-523" (layer "B.Cu")
-    (at 64.29375 88.10625 90)
+    (at 40.48125 88.10625 90)
     (descr "http://www.diodes.com/datasheets/ap02001.pdf p.144")
     (tags "Diode SOD523")
@@
   )
   (footprint "acheron_Connectors:PinHeader_2x5_P2.54mm_Vertical" (layer "B.Cu")
-    (at 208.28 114.3 180)
+    (at 176.2125 138.1125 180)
     (descr "Through hole straight pin header, 1x14, 2.54mm pitch, single row")
     (tags "Through hole pin header THT 1x14 2.54mm single row")
@@
   )
   (footprint "acheron_Connectors:PinHeader_1x4_P2.54mm_Vertical" (layer "B.Cu")
-    (at 214.3125 112.87125 180)
+    (at 183.35625 135.73125 180)
     (descr "Through hole straight pin header, 1x14, 2.54mm pitch, single row")
     (tags "Through hole pin header THT 1x14 2.54mm single row")
@@
   )
   (footprint "Diode_SMD:D_SOD-523" (layer "B.Cu")
-    (at 226.21875 88.10625 90)
+    (at 211.93125 88.10625 90)
     (descr "http://www.diodes.com/datasheets/ap02001.pdf p.144")
     (tags "Diode SOD523")
