File: kicad-files/legshark65_rev2.kicad_sch (KiCad schematic)
At the start: 202 parts, among them J1 ARM JTAG, J2 Conn_01x04, SW1 K2-1187SQ-A4SW-06, SW2 PCM12SMTR, T2 53261-0471, U1 STM32F411CEU6, U2 MCP1700T-3302E/TT, U3 AT24C256C-SSHL-T, Y1 TAXM8M4RFDCET2T

Commit message: Started adding all of the components onto the board
Parts:
- removed J2: Conn_01x04, acheron_Connectors:PinHeader_1x4_P2.54mm_Vertical, symbol Connector_Generic:Conn_01x04
- removed R2, R3: 0R, Resistor_SMD:R_0603_1608Metric, symbol Device:R
Other:
- note removed: "Hardwired alternative"
Changed lines of the file:
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@@
     (stroke (width 0) (type default))
   )
-  (wire (pts (xy 48.26 264.795) (xy 50.165 264.795))
-    (stroke (width 0) (type default))
-  )
   (wire (pts (xy 136.525 123.19) (xy 140.97 123.19))
     (stroke (width 0) (type default))
@@
     (stroke (width 0) (type default))
   )
-  (wire (pts (xy 318.77 24.13) (xy 325.12 24.13))
-    (stroke (width 0) (type default))
+  (polyline (pts (xy 255.905 6.35) (xy 255.905 144.78))
+    (stroke (width 0.5) (type dash))
   )
-  (wire (pts (xy 38.735 264.795) (xy 40.64 264.795))
+  (wire (pts (xy 318.77 24.13) (xy 325.12 24.13))
     (stroke (width 0) (type default))
   )
@@
     (stroke (width 0) (type default))
   )
-  (wire (pts (xy 48.26 262.255) (xy 50.165 262.255))
-    (stroke (width 0) (type default))
-  )
   (wire (pts (xy 186.69 105.41) (xy 186.69 106.68))
     (stroke (width 0) (type default))
@@
     (stroke (width 0) (type default))
   )
-  (wire (pts (xy 47.625 259.715) (xy 50.165 259.715))
-    (stroke (width 0) (type default))
-  )
   (wire (pts (xy 76.2 278.13) (xy 92.71 278.13))
     (stroke (width 0) (type default))
@@
     (stroke (width 0) (type default))
   )
-  (wire (pts (xy 38.735 262.255) (xy 40.64 262.255))
-    (stroke (width 0) (type default))
-  )
   (wire (pts (xy 293.37 123.19) (xy 293.37 125.73))
     (stroke (width 0) (type default))
@@
     (effects (font (size 3 3) (thickness 0.6) bold) (justify right bottom))
   )
-  (text "Hardwired alternative" (at 41.91 256.54 0)
-    (effects (font (size 1.27 1.27)) (justify left bottom))
-  )
   (text "Leave R5 unpopulated as per specs for MCU" (at 236.855 224.155 0)
     (effects (font (size 1.27 1.27)) (justify left bottom))
@@
     )
   )
-  (global_label "D+" (shape bidirectional) (at 38.735 262.255 180) (fields_autoplaced)
-    (effects (font (size 1.27 1.27)) (justify right))
-    (property "Intersheetrefs" "${INTERSHEET_REFS}" (at 32.6885 262.255 0)
-      (effects (font (size 1.27 1.27)) (justify right) hide)
-    )
-  )
   (global_label "row1" (shape input) (at 22.86 60.96 180)
     (effects (font (size 1.27 1.27)) (justify right))
@@
     )
   )
-  (global_label "D-" (shape bidirectional) (at 38.735 264.795 180) (fields_autoplaced)
-    (effects (font (size 1.27 1.27)) (justify right))
-    (property "Intersheetrefs" "${INTERSHEET_REFS}" (at 32.6885 264.795 0)
-      (effects (font (size 1.27 1.27)) (justify right) hide)
-    )
-  )
   (global_label "col5" (shape input) (at 172.72 16.51 180)
     (effects (font (size 1.27 1.27)) (justify right))
@@
     )
   )
-  (global_label "5V" (shape output) (at 50.165 267.335 180) (fields_autoplaced)
-    (effects (font (size 1.27 1.27)) (justify right))
-    (property "Intersheetrefs" "${INTERSHEET_REFS}" (at 45.6153 267.335 0)
-      (effects (font (size 1.27 1.27)) (justify right) hide)
-    )
-  )
   (global_label "col11" (shape input) (at 325.12 16.51 180)
     (effects (font (size 1.27 1.27)) (justify right))
@@
     )
   )
-  (symbol (lib_id "power:GND") (at 47.625 259.715 270) (unit 1)
-    (in_bom yes) (on_board yes) (dnp no)
-    (property "Reference" "#PWR03" (at 41.275 259.715 0)
-      (effects (font (size 1.27 1.27)) hide)
-    )
-    (property "Value" "GND" (at 46.355 257.81 90)
-      (effects (font (size 1.27 1.27)) (justify right))
-    )
-    (property "Footprint" "" (at 47.625 259.715 0)
-      (effects (font (size 1.27 1.27)) hide)
-    )
-    (property "Datasheet" "" (at 47.625 259.715 0)
-      (effects (font (size 1.27 1.27)) hide)
-    )
-    (pin "1")
-    (instances
-      (project "legshark65_rev2"
-        (path "/2fcc1073-d3f4-43f9-b3b4-5cee13272705"
-          (reference "#PWR03") (unit 1)
-        )
-      )
-      (project "old_layout"
-        (path "/2fda2561-53ed-4930-8b41-858e0e3dd5f4"
-          (reference "#PWR031") (unit 1)
-        )
-      )
-      (project "legshark65_rev1"
-        (path "/9ddf6dc5-8b5e-413a-9b25-d1d5a5a60469"
-          (reference "#PWR023") (unit 1)
-        )
-      )
-    )
-  )
   (symbol (lib_id "Device:D_Small") (at 313.69 83.82 90) (unit 1)
     (in_bom yes) (on_board yes) (dnp no)
@@
     )
   )
-  (symbol (lib_id "Connector_Generic:Conn_01x04") (at 55.245 262.255 0) (unit 1)
-    (in_bom yes) (on_board yes) (dnp no) (fields_autoplaced)
-    (property "Reference" "J2" (at 57.785 262.89 0)
-      (effects (font (size 1.27 1.27)) (justify left))
-    )
-    (property "Value" "Conn_01x04" (at 57.785 265.43 0)
-      (effects (font (size 1.27 1.27)) (justify left))
-    )
-    (property "Footprint" "acheron_Connectors:PinHeader_1x4_P2.54mm_Vertical" (at 55.245 262.255 0)
-      (effects (font (size 1.27 1.27)) hide)
-    )
-    (property "Datasheet" "~" (at 55.245 262.255 0)
-      (effects (font (size 1.27 1.27)) hide)
-    )
-    (pin "1")
-    (pin "2")
-    (pin "3")
-    (pin "4")
-    (instances
-      (project "legshark65_rev2"
-        (path "/2fcc1073-d3f4-43f9-b3b4-5cee13272705"
-          (reference "J2") (unit 1)
-        )
-      )
-      (project "legshark65_rev1"
-        (path "/9ddf6dc5-8b5e-413a-9b25-d1d5a5a60469"
-          (reference "J2") (unit 1)
-        )
-      )
-    )
-  )
   (symbol (lib_id "Memory_EEPROM:24LC256") (at 187.96 162.56 180) (unit 1)
     (in_bom yes) (on_board yes) (dnp no)
@@
     )
   )
-  (symbol (lib_id "Device:R") (at 44.45 262.255 270) (mirror x) (unit 1)
-    (in_bom yes) (on_board yes) (dnp no)
-    (property "Reference" "R2" (at 42.545 260.35 90)
-      (effects (font (size 1.27 1.27)))
-    )
-    (property "Value" "0R" (at 44.45 262.255 90)
-      (effects (font (size 1.27 1.27)))
-    )
-    (property "Footprint" "Resistor_SMD:R_0603_1608Metric" (at 44.45 264.033 90)
-      (effects (font (size 1.27 1.27)) hide)
-    )
-    (property "Datasheet" "~" (at 44.45 262.255 0)
-      (effects (font (size 1.27 1.27)) hide)
-    )
-    (property "Description" "UNPOPULATE" (at 44.45 262.255 0)
-      (effects (font (size 1.27 1.27)) hide)
-    )
-    (pin "1")
-    (pin "2")
-    (instances
-      (project "legshark65_rev2"
-        (path "/2fcc1073-d3f4-43f9-b3b4-5cee13272705"
-          (reference "R2") (unit 1)
-        )
-      )
-      (project "old_layout"
-        (path "/2fda2561-53ed-4930-8b41-858e0e3dd5f4"
-          (reference "R5") (unit 1)
-        )
-      )
-      (project "legshark65_rev1"
-        (path "/9ddf6dc5-8b5e-413a-9b25-d1d5a5a60469"
-          (reference "R3") (unit 1)
-        )
-      )
-    )
-  )
   (symbol (lib_id "Device:D_Small") (at 212.09 109.22 90) (unit 1)
     (in_bom yes) (on_board yes) (dnp no)
@@
         )
       )
-    )
-  )
-  (symbol (lib_id "Device:R") (at 44.45 264.795 270) (mirror x) (unit 1)
-    (in_bom yes) (on_board yes) (dnp no)
-    (property "Reference" "R3" (at 43.18 266.7 90)
-      (effects (font (size 1.27 1.27)))
-    )
-    (property "Value" "0R" (at 44.45 264.795 90)
-      (effects (font (size 1.27 1.27)))
-    )
-    (property "Footprint" "Resistor_SMD:R_0603_1608Metric" (at 44.45 266.573 90)
-      (effects (font (size 1.27 1.27)) hide)
-    )
-    (property "Datasheet" "~" (at 44.45 264.795 0)
-      (effects (font (size 1.27 1.27)) hide)
-    )
-    (property "Description" "UNPOPULATE" (at 44.45 264.795 0)
-      (effects (font (size 1.27 1.27)) hide)
-    )
-    (pin "1")
-    (pin "2")
-    (instances
-      (project "legshark65_rev2"
-        (path "/2fcc1073-d3f4-43f9-b3b4-5cee13272705"
-          (reference "R3") (unit 1)
-        )
-      )
-      (project "old_layout"
-        (path "/2fda2561-53ed-4930-8b41-858e0e3dd5f4"
-          (reference "R5") (unit 1)
-        )
-      )
-      (project "legshark65_rev1"
-        (path "/9ddf6dc5-8b5e-413a-9b25-d1d5a5a60469"
-          (reference "R2") (unit 1)
-        )
-      )

Commit message: Started running some test routes
Connections:
- net 3V3: no longer J1.7 (Pin_7), J1.8 (Pin_8)
- net BOOT0: no longer J1.5 (Pin_5)
- net BOOT1: no longer J1.6 (Pin_6)
- net GND: now also C1.1; no longer C1.2, J1.10 (Pin_10), J1.3 (Pin_3), J1.4 (Pin_4)
- net NRST: no longer J1.9 (Pin_9)
- net SWCLK: no longer J1.2 (Pin_2)
- net SWDIO: no longer J1.1 (Pin_1)
- net at U1.6 (PD1/OSC_OUT), Y1.3: now also C1.2; no longer C1.1
Other:
- moved on the sheet: C1, J1
Changed lines of the file:
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@@
     )
   )
-  (symbol (lib_id "Connector_Generic:Conn_02x05_Odd_Even") (at 50.165 213.36 0) (unit 1)
-    (in_bom yes) (on_board yes) (dnp no) (fields_autoplaced)
-    (property "Reference" "J1" (at 51.435 202.565 0)
+  (symbol (lib_id "Connector_Generic:Conn_02x05_Odd_Even") (at 50.165 213.36 0) (mirror y) (unit 1)
+    (in_bom yes) (on_board yes) (dnp no)
+    (property "Reference" "J1" (at 48.895 202.565 0)
       (effects (font (size 1.27 1.27)))
     )
-    (property "Value" "ARM JTAG" (at 51.435 205.105 0)
+    (property "Value" "ARM JTAG" (at 48.895 205.105 0)
       (effects (font (size 1.27 1.27)))
     )
@@
     )
   )
-  (symbol (lib_id "Device:C") (at 100.33 236.22 90) (unit 1)
-    (in_bom yes) (on_board yes) (dnp no)
-    (property "Reference" "C1" (at 99.06 240.03 90)
+  (symbol (lib_id "Device:C") (at 100.33 236.22 270) (mirror x) (unit 1)
+    (in_bom yes) (on_board yes) (dnp no)
+    (property "Reference" "C1" (at 101.6 240.03 90)
       (effects (font (size 1.27 1.27)) (justify left))
     )
-    (property "Value" "15p" (at 104.14 240.03 90)
+    (property "Value" "15p" (at 96.52 240.03 90)
       (effects (font (size 1.27 1.27)) (justify left))
     )
-    (property "Footprint" "Capacitor_SMD:C_0603_1608Metric_Pad1.08x0.95mm_HandSolder" (at 104.14 235.2548 0)
-      (effects (font (size 1.27 1.27)) hide)
-    )
+    (property "Footprint" "Capacitor_SMD:C_0603_1608Metric_Pad1.08x0.95mm_HandSolder" (at 96.52 235.2548 0)
+      (effects (font (size 1.27 1.27)) hide)
+    )

Commit message: Added more routing and planning
Connections:
- net 3V3: now also J1.7 (Pin_7), J1.8 (Pin_8)
- net BOOT0: now also J1.6 (Pin_6)
- net BOOT1: now also J1.5 (Pin_5)
- net D+: now also T2.3 (D+); no longer T2.2 (D-)
- net D-: now also T2.2 (D-); no longer T2.3 (D+)
- net GND: now also J1.3 (Pin_3), J1.4 (Pin_4), J1.9 (Pin_9)
- net NRST: now also J1.10 (Pin_10)
- net SWCLK: now also J1.1 (Pin_1)
- net SWDIO: now also J1.2 (Pin_2)
Changed lines of the file:
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@@
     )
   )
-  (global_label "BOOT1" (shape input) (at 57.785 213.36 0) (fields_autoplaced)
+  (global_label "BOOT1" (shape input) (at 55.245 213.36 0) (fields_autoplaced)
     (effects (font (size 1.27 1.27)) (justify left))
-    (property "Intersheetrefs" "${INTERSHEET_REFS}" (at 66.1447 213.36 0)
+    (property "Intersheetrefs" "${INTERSHEET_REFS}" (at 63.6047 213.36 0)
       (effects (font (size 1.27 1.27)) (justify left) hide)
     )
@@
     )
   )
-  (global_label "D-" (shape bidirectional) (at 49.53 232.41 90) (fields_autoplaced)
+  (global_label "D-" (shape bidirectional) (at 53.34 232.41 90) (fields_autoplaced)
     (effects (font (size 1.27 1.27)) (justify left))
-    (property "Intersheetrefs" "${INTERSHEET_REFS}" (at 49.53 226.3635 90)
+    (property "Intersheetrefs" "${INTERSHEET_REFS}" (at 53.34 226.3635 90)
       (effects (font (size 1.27 1.27)) (justify left) hide)
     )
@@
     )
   )
-  (global_label "NRST" (shape input) (at 45.085 218.44 180) (fields_autoplaced)
+  (global_label "NRST" (shape input) (at 42.545 218.44 180) (fields_autoplaced)
     (effects (font (size 1.27 1.27)) (justify right))
-    (property "Intersheetrefs" "${INTERSHEET_REFS}" (at 38.0558 218.44 0)
+    (property "Intersheetrefs" "${INTERSHEET_REFS}" (at 35.5158 218.44 0)
       (effects (font (size 1.27 1.27)) (justify right) hide)
     )
@@
     )
   )
-  (global_label "3V3" (shape input) (at 45.085 215.9 180) (fields_autoplaced)
+  (global_label "3V3" (shape input) (at 42.545 215.9 180) (fields_autoplaced)
     (effects (font (size 1.27 1.27)) (justify right))
-    (property "Intersheetrefs" "${INTERSHEET_REFS}" (at 39.3258 215.9 0)
+    (property "Intersheetrefs" "${INTERSHEET_REFS}" (at 36.7858 215.9 0)
       (effects (font (size 1.27 1.27)) (justify right) hide)
     )
@@
     )
   )
-  (global_label "3V3" (shape input) (at 57.785 215.9 0) (fields_autoplaced)
+  (global_label "3V3" (shape input) (at 55.245 215.9 0) (fields_autoplaced)
     (effects (font (size 1.27 1.27)) (justify left))
-    (property "Intersheetrefs" "${INTERSHEET_REFS}" (at 63.5442 215.9 0)
+    (property "Intersheetrefs" "${INTERSHEET_REFS}" (at 61.0042 215.9 0)
       (effects (font (size 1.27 1.27)) (justify left) hide)
     )
   )
-  (global_label "D+" (shape bidirectional) (at 53.34 232.41 90) (fields_autoplaced)
+  (global_label "D+" (shape bidirectional) (at 49.53 232.41 90) (fields_autoplaced)
     (effects (font (size 1.27 1.27)) (justify left))
-    (property "Intersheetrefs" "${INTERSHEET_REFS}" (at 53.34 226.3635 90)
+    (property "Intersheetrefs" "${INTERSHEET_REFS}" (at 49.53 226.3635 90)
       (effects (font (size 1.27 1.27)) (justify left) hide)
     )
   )
-  (global_label "BOOT0" (shape input) (at 45.085 213.36 180) (fields_autoplaced)
+  (global_label "BOOT0" (shape input) (at 42.545 213.36 180) (fields_autoplaced)
     (effects (font (size 1.27 1.27)) (justify right))
-    (property "Intersheetrefs" "${INTERSHEET_REFS}" (at 36.7253 213.36 0)
+    (property "Intersheetrefs" "${INTERSHEET_REFS}" (at 34.1853 213.36 0)
       (effects (font (size 1.27 1.27)) (justify right) hide)
     )
@@
     )
   )
-  (global_label "SWDIO" (shape input) (at 45.085 208.28 180) (fields_autoplaced)
+  (global_label "SWDIO" (shape input) (at 42.545 208.28 180) (fields_autoplaced)
     (effects (font (size 1.27 1.27)) (justify right))
-    (property "Intersheetrefs" "${INTERSHEET_REFS}" (at 36.9672 208.28 0)
+    (property "Intersheetrefs" "${INTERSHEET_REFS}" (at 34.4272 208.28 0)
       (effects (font (size 1.27 1.27)) (justify right) hide)
     )
@@
     )
   )
-  (global_label "SWCLK" (shape input) (at 57.785 208.28 0) (fields_autoplaced)
+  (global_label "SWCLK" (shape input) (at 55.245 208.28 0) (fields_autoplaced)
     (effects (font (size 1.27 1.27)) (justify left))
-    (property "Intersheetrefs" "${INTERSHEET_REFS}" (at 66.2656 208.28 0)
+    (property "Intersheetrefs" "${INTERSHEET_REFS}" (at 63.7256 208.28 0)
       (effects (font (size 1.27 1.27)) (justify left) hide)
     )
@@
     )
   )
-  (symbol (lib_id "power:GND") (at 57.785 218.44 90) (unit 1)
+  (symbol (lib_id "power:GND") (at 55.245 218.44 90) (unit 1)
     (in_bom yes) (on_board yes) (dnp no)
-    (property "Reference" "#PWR06" (at 64.135 218.44 0)
+    (property "Reference" "#PWR06" (at 61.595 218.44 0)
       (effects (font (size 1.27 1.27)) hide)
     )
-    (property "Value" "GND" (at 61.595 218.44 0)
+    (property "Value" "GND" (at 59.055 218.44 0)
       (effects (font (size 1.27 1.27)))
     )
-    (property "Footprint" "" (at 57.785 218.44 0)
+    (property "Footprint" "" (at 55.245 218.44 0)
       (effects (font (size 1.27 1.27)) hide)
     )
-    (property "Datasheet" "" (at 57.785 218.44 0)
+    (property "Datasheet" "" (at 55.245 218.44 0)
       (effects (font (size 1.27 1.27)) hide)
     )
@@
     )
   )
-  (symbol (lib_id "power:GND") (at 57.785 210.82 90) (unit 1)
+  (symbol (lib_id "power:GND") (at 55.245 210.82 90) (unit 1)
     (in_bom yes) (on_board yes) (dnp no)
-    (property "Reference" "#PWR05" (at 64.135 210.82 0)
+    (property "Reference" "#PWR05" (at 61.595 210.82 0)
       (effects (font (size 1.27 1.27)) hide)
     )
-    (property "Value" "GND" (at 61.595 210.82 0)
+    (property "Value" "GND" (at 59.055 210.82 0)
       (effects (font (size 1.27 1.27)))
     )
-    (property "Footprint" "" (at 57.785 210.82 0)
+    (property "Footprint" "" (at 55.245 210.82 0)
       (effects (font (size 1.27 1.27)) hide)
     )
-    (property "Datasheet" "" (at 57.785 210.82 0)
+    (property "Datasheet" "" (at 55.245 210.82 0)
       (effects (font (size 1.27 1.27)) hide)
     )
@@
     )
   )
-  (symbol (lib_id "power:GND") (at 45.085 210.82 270) (unit 1)
+  (symbol (lib_id "power:GND") (at 42.545 210.82 270) (unit 1)
     (in_bom yes) (on_board yes) (dnp no)
-    (property "Reference" "#PWR01" (at 38.735 210.82 0)
+    (property "Reference" "#PWR01" (at 36.195 210.82 0)
       (effects (font (size 1.27 1.27)) hide)
     )
-    (property "Value" "GND" (at 41.275 210.82 0)
+    (property "Value" "GND" (at 38.735 210.82 0)
       (effects (font (size 1.27 1.27)))
     )
-    (property "Footprint" "" (at 45.085 210.82 0)
+    (property "Footprint" "" (at 42.545 210.82 0)
       (effects (font (size 1.27 1.27)) hide)
     )
-    (property "Datasheet" "" (at 45.085 210.82 0)
+    (property "Datasheet" "" (at 42.545 210.82 0)
       (effects (font (size 1.27 1.27)) hide)
     )
